Commit message: andre commit fikset joint bevegelse

File: src/moonmapper_description/urdf/moonmapper_rover.urdf.xacro (robot description, xacro)
@@ -4,4 +4,7 @@
   <xacro:property name="deg" value="0.017453292519943295"/> <!-- pi/180 -->
   <!-- NOTE: Keeping this file argument-free for simple launching. -->
+  <!-- URDF mimic-tagging is intended ONLY for RViz / kinematic visualization.
+       In Gazebo, mimic can fight physics constraints / plugins and stiffen the suspension. -->
+  <xacro:arg name="enable_urdf_mimic" default="true"/>
   <!-- Base footprint frame for RViz / navigation stacks -->
   <link name="base_footprint"/>
@@ -23,8 +26,10 @@
     </visual>
     <collision>
-      <origin xyz="0 0 0" rpy="0 0 0"/>
-      <geometry>
-        <mesh filename="package://moonmapper_description/meshes/visual/robot_base.stl"
-              scale="1 1 1"/>
+      <!-- Stabil sim-collision: primitiv boks i stedet for detaljert STL.
+           Hindrer at skarpe detaljer tar bakken og “tipper” roveren før
+           rocker/bogie får jobbe. Størrelse fra notat i filen: 48x25x18mm. -->
+      <origin xyz="0 0 0" rpy="0 0 0"/>
+      <geometry>
+        <box size="0.048 0.025 0.018"/>
       </geometry>
     </collision>
@@ -49,9 +54,9 @@
          - wheel_[lr][123]_joint (continuous, Y)
        Feste-braketten + mellomstykket + stang er STIV-SVEISET til rockeren
-       (fixed). Dette er fysisk korrekt: push-arm-strukturen paa toppen av
+       (fixed). Dette er fysisk korrekt: push-arm-strukturen på toppen av
        en rocker har ingen egen frihetsgrad relativt til rockeren.
        Den lukkede sloeyfen mellom stang-tuppen og diff-staven i chassiset
-       lar seg IKKE representere i URDF (trestruktur). Vi loeser det ved:
-         * RViz: mimic-tagger paa rocker_left_joint og rocker_bogie_diff_joint
+       lar seg IKKE representere i URDF (trestruktur). Vi løser det ved:
+         * RViz: mimic-tagger på rocker_left_joint og rocker_bogie_diff_joint
          * Gazebo: RockerBogieDifferential-pluginen (PD-constraint)
        ===================================================================== -->
@@ -59,5 +64,5 @@
        HOEYRE SIDE
        ===================================================================== -->
-  <!-- Rocker (revolute) festet direkte paa chassiset.
+  <!-- Rocker (revolute) festet direkte på chassiset.
        Origin = gammel "feste_rocker_bogie" fixed-offset + gammel rocker-offset:
          (0.014227,-0.065999,0.021756) + (-0.013717,-0.001277,-0.007986)
@@ -97,5 +102,5 @@
     <axis xyz="0 1 0"/>
     <dynamics damping="0.02" friction="0.005"/>
-    <limit lower="${-30*deg}" upper="${30*deg}" effort="100" velocity="2.0"/>
+    <limit lower="-0.133" upper="0.133" effort="100" velocity="6.0"/>
   </joint>
   <!-- Mellomstykket er sveiset fast i toppen av braketten. -->
@@ -119,8 +124,13 @@
     </inertial>
   </link>
-  <joint name="feste_mellom_feste_og_stang_right_joint" type="fixed">
-    <parent link="rocker_right_link"/>
+  <joint name="feste_mellom_feste_og_stang_right_joint" type="prismatic">
+    <parent link="base_link"/>
     <child link="feste_mellom_feste_og_stang_right_link"/>
-    <origin xyz="-0.006290 -0.001307 0.054591" rpy="0 0 0"/>
+    <origin xyz="0.013913 -0.067245 0.076373" rpy="0 0 0"/>
+    <axis xyz="1 0 0"/>
+    <xacro:if value="$(arg enable_urdf_mimic)">
+      <mimic joint="rocker_bogie_diff_joint" multiplier="0.05" offset="0.0"/>
+    </xacro:if>
+     <limit lower="${-1*deg}" upper="${1*deg}" effort="50" velocity="3.0"/>
   </joint>
   <!-- Staget er sveiset fast i mellomstykket. Tupp-enden som fysisk skal
@@ -146,8 +156,13 @@
     </inertial>
   </link>
-  <joint name="stang_right_joint" type="fixed">
+  <joint name="stang_right_joint" type="prismatic">
     <parent link="feste_mellom_feste_og_stang_right_link"/>
     <child link="stang_right_link"/>
-    <origin xyz="-0.095753 -0.000079 0.000059" rpy="0 0 0"/>
+    <origin xyz="-0.101730 -0.000140 0.000033" rpy="0 0 0"/>
+    <axis xyz="1 0 0"/>
+    <xacro:if value="$(arg enable_urdf_mimic)">
+      <mimic joint="feste_mellom_feste_og_stang_right_joint" multiplier="0.05" offset="0.0"/>
+    </xacro:if>
+    <limit lower="${-1*deg}" upper="${1*deg}" effort="50" velocity="3.0"/>
   </joint>
   <!-- Bogie (revolute, Y) parentet paa ROCKEREN, ikke paa braketten.
@@ -189,5 +204,5 @@
     <axis xyz="0 1 0"/>
     <dynamics damping="0.01" friction="0.003"/>
-    <limit lower="${-40*deg}" upper="${40*deg}" effort="100" velocity="2.0"/>
+    <limit lower="${-40*deg}" upper="${40*deg}" effort="100" velocity="6.0"/>
   </joint>
   <!-- Hoeyre hjul: r1 paa rocker, r2+r3 paa bogie. Continuous (ingen limits). -->
@@ -403,6 +418,8 @@
     <axis xyz="0 1 0"/>
     <dynamics damping="0.02" friction="0.005"/>
-    <limit lower="${-30*deg}" upper="${30*deg}" effort="100" velocity="2.0"/>
+    <limit lower="-0.133" upper="0.133" effort="100" velocity="6.0"/>
+    <xacro:if value="$(arg enable_urdf_mimic)">
       <mimic joint="rocker_right_joint" multiplier="-1.0" offset="0.0"/>
+    </xacro:if>
   </joint>
   <link name="feste_mellom_feste_og_stang_left_link">
@@ -425,8 +442,13 @@
     </inertial>
   </link>
-  <joint name="feste_mellom_feste_og_stang_left_joint" type="fixed">
-    <parent link="rocker_left_link"/>
+  <joint name="feste_mellom_feste_og_stang_left_joint" type="prismatic">
+    <parent link="base_link"/>
     <child link="feste_mellom_feste_og_stang_left_link"/>
-    <origin xyz="-0.006425 0.001235 0.054592" rpy="0 0 0"/>
+    <origin xyz="0.013977 0.064006 0.076371" rpy="0 0 0"/>
+    <xacro:if value="$(arg enable_urdf_mimic)">
+      <mimic joint="rocker_bogie_diff_joint" multiplier="0.05" offset="0.0"/>
+    </xacro:if>
+    <axis xyz="1 0 0"/>
+    <limit lower="${-1*deg}" upper="${1*deg}" effort="50" velocity="3.0"/>
   </joint>
   <link name="stang_left_link">
@@ -449,8 +471,13 @@
     </inertial>
   </link>
-  <joint name="stang_left_joint" type="fixed">
+  <joint name="stang_left_joint" type="prismatic">
     <parent link="feste_mellom_feste_og_stang_left_link"/>
     <child link="stang_left_link"/>
-    <origin xyz="-0.095753 -0.000079 0.000059" rpy="0 0 0"/>
+    <origin xyz="-0.101903 0.001198 0.000110" rpy="0 0 0"/>
+    <axis xyz="1 0 0"/>
+    <xacro:if value="$(arg enable_urdf_mimic)">
+      <mimic joint="feste_mellom_feste_og_stang_left_joint" multiplier="0.05" offset="0.0"/>
+    </xacro:if>
+    <limit lower="${-1*deg}" upper="${1*deg}" effort="50" velocity="3.0"/>
   </joint>
   <!-- Bogie venstre. Origin = (0.013707,0.001287,-0.008001)-(-0.013851,0.001264,-0.007984)
@@ -488,5 +515,5 @@
     <axis xyz="0 1 0"/>
     <dynamics damping="0.01" friction="0.003"/>
-    <limit lower="${-40*deg}" upper="${40*deg}" effort="100" velocity="2.0"/>
+    <limit lower="${-40*deg}" upper="${40*deg}" effort="100" velocity="6.0"/>
   </joint>
   <!-- Venstre hjul: l1 paa rocker, l2+l3 paa bogie. Continuous (ingen limits). -->
@@ -754,4 +781,58 @@
   </inertial>
 </link>
+<!-- ===============================================================
+     VISUELL "TIP"-GEOMETRI FOR PUSHRODS VED DIFF-BEAM
+     URDF kan ikke representere den lukkede løkken (stang-tupp <-> beam-ende).
+     For å unngå at stang_endene ser ut som de "stikker ut", legger vi inn
+     to små endebeslag som er barn av diff-beamet. Disse følger diffens yaw
+     (rocker_bogie_diff_joint), slik at den visuelle mekanikken ser korrekt ut
+     selv om den fysiske koblingen håndheves av pluginen via rocker-constraint.
+     Plassering bruker samme halvlengde som dokumentert i diff-kommentaren:
+       diff-stav halvlengde ≈ 0.0747 m langs Y i diff-link frame.
+     =============================================================== -->
+<link name="stang_left_tip_link">
+  <!-- Bruk primitiv visual her: mesh-filene hengsel_diff_* finnes ikke i
+       moonmapper_description/meshes/visual i denne repo-versjonen. -->
+  <visual>
+    <origin xyz="0 0 0" rpy="0 0 0"/>
+    <geometry>
+      <sphere radius="0.004"/>
+    </geometry>
+    <material name="moonmapper_dark_gray">
+      <color rgba="0.35 0.35 0.35 1.0"/>
+    </material>
+  </visual>
+  <inertial>
+    <origin xyz="0 0 0" rpy="0 0 0"/>
+    <mass value="0.001"/>
+    <inertia ixx="1e-8" ixy="0" ixz="0" iyy="1e-8" iyz="0" izz="1e-8"/>
+  </inertial>
+</link>
+<joint name="stang_left_tip_joint" type="fixed">
+  <parent link="rocker_bogie_diff_link"/>
+  <child link="stang_left_tip_link"/>
+  <origin xyz="0.0 0.0747 0.0" rpy="0 0 0"/>
+</joint>
+<link name="stang_right_tip_link">
+  <visual>
+    <origin xyz="0 0 0" rpy="0 0 0"/>
+    <geometry>
+      <sphere radius="0.004"/>
+    </geometry>
+    <material name="moonmapper_dark_gray">
+      <color rgba="0.35 0.35 0.35 1.0"/>
+    </material>
+  </visual>
+  <inertial>
+    <origin xyz="0 0 0" rpy="0 0 0"/>
+    <mass value="0.001"/>
+    <inertia ixx="1e-8" ixy="0" ixz="0" iyy="1e-8" iyz="0" izz="1e-8"/>
+  </inertial>
+</link>
+<joint name="stang_right_tip_joint" type="fixed">
+  <parent link="rocker_bogie_diff_link"/>
+  <child link="stang_right_tip_link"/>
+  <origin xyz="0.0 -0.0747 0.0" rpy="0 0 0"/>
+</joint>
 <!-- Walking-beam staven paa toppen av chassiset.
      Kinematisk utledning (virtuelt ball-link mellom push-arm-tupp og stav-ende):
@@ -768,7 +849,14 @@
   <origin xyz="0.000012 0.000001 0.014" rpy="0 0 0"/>
   <axis xyz="0 0 1"/>
-  <dynamics damping="0.8" friction="0.08"/>
-  <limit lower="${-90*deg}" upper="${90*deg}" effort="100" velocity="2.0"/>
+  <!-- Diff-staven er en lett, kosmetisk link som PD-drives i Gazebo.
+       Høy URDF-damping/friction her kan låse hele rocker-systemet indirekte.
+       Hold den derfor myk; stabilisering skjer i pluginens PD-gains. -->
+  <dynamics damping="0.02" friction="0.002"/>
+  <!-- Ikke la diff-leddet mettes på lav velocity-limit; det er en "kosmetisk"
+       ledd som må kunne følge pluginens target uten å klippe hastigheten. -->
+  <limit lower="${-90*deg}" upper="${90*deg}" effort="100" velocity="10.0"/>
+  <xacro:if value="$(arg enable_urdf_mimic)">
     <mimic joint="rocker_right_joint" multiplier="0.82" offset="0.0"/>
+  </xacro:if>
 </joint>
 <!-- === Tak (skroghette over kjernen av chassiset) === -->

File: src/moonmapper_description/urdf/moonmapper_rover_gazebo.urdf.xacro (robot description, xacro)
@@ -3,4 +3,21 @@
   <!-- Grunnmodell: samme fil som RViz bruker -->
   <xacro:include filename="$(find moonmapper_description)/urdf/moonmapper_rover.urdf.xacro"/>
+  <!-- Slå av tunge/verbose plugins under suspension-debug -->
+  <xacro:arg name="enable_triad_spectroscopy" default="true"/>
+  <!-- Diff-plugin tuning (eksponeres som launch-args) -->
+  <!-- right_sign=+1 => err=qL+qR. right_sign=-1 => err=qL-qR.
+       I praksis velger vi verdien som IKKE metter rockerne i joint-limits ved hvile. -->
+  <xacro:arg name="diff_right_sign" default="1.0"/>
+  <xacro:arg name="diff_kp" default="5.0"/>
+  <xacro:arg name="diff_kd" default="0.5"/>
+  <xacro:arg name="diff_max_torque" default="0.5"/>
+  <xacro:arg name="diff_k_diff_L" default="-0.41"/>
+  <xacro:arg name="diff_k_diff_R" default="0.41"/>
+  <xacro:arg name="diff_k_diff_0" default="0.0"/>
+  <!-- Aux-PD er "kosmetisk" men påvirker stabilitet hvis den metter og slår i velocity-limit.
+       Vi velger derfor litt lavere kp, høyere kd og moderat max torque. -->
+  <xacro:arg name="diff_kp_aux" default="0.8"/>
+  <xacro:arg name="diff_kd_aux" default="0.4"/>
+  <xacro:arg name="diff_max_torque_aux" default="0.12"/>
   <!-- Kontakt/friksjons-parametere for hjul. mu1/mu2 er relativt hoeye fordi
        hjul-masse er kun ~0.02 kg pr hjul; lav friksjon ville gi sludging paa
@@ -35,16 +52,18 @@
        ikke daglige svingninger loese naar ingen styrer dem) -->
   <gazebo reference="rocker_left_joint">
-    <implicitSpringDamper>true</implicitSpringDamper>
+    <!-- implicitSpringDamper kan i praksis introdusere en "skjult" fjær som gjør
+         passive joints kunstig stive i enkelte physics-backends. Hold dette av. -->
+    <implicitSpringDamper>false</implicitSpringDamper>
     <provideFeedback>true</provideFeedback>
   </gazebo>
   <gazebo reference="rocker_right_joint">
-    <implicitSpringDamper>true</implicitSpringDamper>
+    <implicitSpringDamper>false</implicitSpringDamper>
     <provideFeedback>true</provideFeedback>
   </gazebo>
   <gazebo reference="bogie_left_joint">
-    <implicitSpringDamper>true</implicitSpringDamper>
+    <implicitSpringDamper>false</implicitSpringDamper>
   </gazebo>
   <gazebo reference="bogie_right_joint">
-    <implicitSpringDamper>true</implicitSpringDamper>
+    <implicitSpringDamper>false</implicitSpringDamper>
   </gazebo>
   <!-- Diff-staven er den eneste revolute joint paa top-linkage-siden.
@@ -52,5 +71,5 @@
        affin funksjon av rocker-vinkene. -->
   <gazebo reference="rocker_bogie_diff_joint">
-    <implicitSpringDamper>true</implicitSpringDamper>
+    <implicitSpringDamper>false</implicitSpringDamper>
     <provideFeedback>true</provideFeedback>
   </gazebo>
@@ -131,8 +150,16 @@
       <hengsel_right_joint></hengsel_right_joint>
       <!-- Primaer-PD: sum-constraint paa rockerne (walking-beam). -->
-      <kp>2.0</kp>
-      <kd>0.2</kd>
+      <!-- Strammere constraint: roveren er lett, og terrengkontakt lager korte
+           impulser; for lav kp/max_torque gjør at walking-beam-effekten uteblir. -->
+      <kp>$(arg diff_kp)</kp>
+      <kd>$(arg diff_kd)</kd>
       <target_sum>0.0</target_sum>
-      <max_torque>0.2</max_torque>
+      <max_torque>$(arg diff_max_torque)</max_torque>
+      <!-- Fortegn for hoeyre side i constrainten:
+           err = qL + right_sign*qR - target_sum
+           Default +1.0 tilsvarer qL + qR = 0.
+           Sett -1.0 hvis hoeyre joint sin positive retning er speilet. -->
+      <!-- err = qL + right_sign*qR - target_sum -->
+      <right_sign>$(arg diff_right_sign)</right_sign>
       <!-- Kinematikk for diff-staven:
              q_diff* = k_diff_L*qL + k_diff_R*qR + k_diff_0
@@ -140,10 +167,17 @@
              q_diff* = 0.82*qR  ->  k_diff_L=0, k_diff_R=0.82           Snu fortegn paa k_diff_R hvis staven dreier motsatt av rockeren. -->
       <k_diff_L>0.0</k_diff_L>
-      <k_diff_R>0.82</k_diff_R>
-      <k_diff_0>0.0</k_diff_0>
-      <!-- Aux-PD: diff-staven er ~5g, så gainene er svært lave. -->
-      <kp_aux>0.2</kp_aux>
-      <kd_aux>0.02</kd_aux>
-      <max_torque_aux>0.02</max_torque_aux>
+      <!-- Diff-beam yaw bør avhenge av BEGGE rockere:
+           Ved symmetri (qL=-qR) ønsker vi fortsatt q_diff* ≈ 0.82*qR.
+           Dette oppnås med: q_diff* = 0.41*(qR - qL). -->
+      <k_diff_L>$(arg diff_k_diff_L)</k_diff_L>
+      <k_diff_R>$(arg diff_k_diff_R)</k_diff_R>
+      <k_diff_0>$(arg diff_k_diff_0)</k_diff_0>
+      <!-- Aux-PD (diff-ledd): i praksis må dette være sterkt nok til å overvinne
+           friksjon, solver-demping og numerikk. For lavt moment her gjør at
+           rocker_bogie_diff_joint ser "låst" ut selv om pluginen kjører. -->
+      <!-- Aux-PD (diff-ledd): nok moment til å følge target uten å mettes på velocity limit. -->
+      <kp_aux>$(arg diff_kp_aux)</kp_aux>
+      <kd_aux>$(arg diff_kd_aux)</kd_aux>
+      <max_torque_aux>$(arg diff_max_torque_aux)</max_torque_aux>
     </plugin>
     </xacro:if>
@@ -163,17 +197,19 @@
     <!-- Level 1: Synthetic Triad spectroscopy sensors (raycast)    -->
     <!-- ========================================================= -->
-    <plugin filename="libmoonmapper_triad_spectroscopy.so"
-            name="moonmapper::TriadSpectroscopy">
-      <enable>true</enable>
-      <update_rate_hz>20</update_rate_hz>
-      <max_distance>0.12</max_distance>
-      <noise_stddev>0.02</noise_stddev>
-      <channels>18</channels>
-      <sensor1_link>triad_sensor_1_link</sensor1_link>
-      <sensor2_link>triad_sensor_2_link</sensor2_link>
-      <topic1>/triad_sensor_1/spectrum</topic1>
-      <topic2>/triad_sensor_2/spectrum</topic2>
-      <material_map_yaml>$(find moonmapper_gz_sensors)/config/triad_material_map.yaml</material_map_yaml>
-    </plugin>
+    <xacro:if value="$(arg enable_triad_spectroscopy)">
+      <plugin filename="libmoonmapper_triad_spectroscopy.so"
+              name="moonmapper::TriadSpectroscopy">
+        <enable>true</enable>
+        <update_rate_hz>20</update_rate_hz>
+        <max_distance>0.12</max_distance>
+        <noise_stddev>0.02</noise_stddev>
+        <channels>18</channels>
+        <sensor1_link>triad_sensor_1_link</sensor1_link>
+        <sensor2_link>triad_sensor_2_link</sensor2_link>
+        <topic1>/triad_sensor_1/spectrum</topic1>
+        <topic2>/triad_sensor_2/spectrum</topic2>
+        <material_map_yaml>$(find moonmapper_gz_sensors)/config/triad_material_map.yaml</material_map_yaml>
+      </plugin>
+    </xacro:if>
   </gazebo>
   <!-- =============================================================== -->
