Commit message: Fix stable 6WD Gazebo physics and motion tests

File: src/moonmapper_description/urdf/moonmapper_rover.urdf.xacro (robot description, xacro)
@@ -9,5 +9,5 @@
   <xacro:arg name="enable_urdf_mimic" default="true"/>
   <xacro:arg name="use_gazebo" default="false"/>
-  <!-- Enkle primitiver for rocker/bogie i stedet for STL (mindre «krok» mot bakken). Hjul bruker alltid sylinder-kollisjon. -->
+  <!-- simple_collision_debug: kun hjul har kollisjon (ingen rocker/bogie/diff-bar) — anbefalt for Gazebo 6WD-traksjon. -->
   <xacro:arg name="simple_collision_debug" default="false"/>
   <xacro:macro name="rocker_stl_collision" params="mesh_file">
@@ -20,8 +20,9 @@
   </xacro:macro>
   <xacro:macro name="rocker_primitive_collision">
+  <!-- Raised/shrunk vs full STL: unngår at rocker-boks treffer regolith før hjulene (slip ved rotasjon). -->
     <collision>
-      <origin xyz="0 0 0" rpy="0 0 0"/>
-      <geometry>
-        <box size="0.16 0.042 0.042"/>
+      <origin xyz="0 0.010 0" rpy="0 0 0"/>
+      <geometry>
+        <box size="0.14 0.034 0.034"/>
       </geometry>
     </collision>
@@ -29,7 +30,7 @@
   <xacro:macro name="bogie_primitive_collision">
     <collision>
-      <origin xyz="0 0 0" rpy="0 0 0"/>
-      <geometry>
-        <box size="0.12 0.052 0.052"/>
+      <origin xyz="0 0.014 0" rpy="0 0 0"/>
+      <geometry>
+        <box size="0.10 0.040 0.028"/>
       </geometry>
     </collision>
@@ -100,7 +101,4 @@
       </material>
     </visual>
-    <xacro:if value="$(arg simple_collision_debug)">
-      <xacro:rocker_primitive_collision/>
-    </xacro:if>
     <xacro:unless value="$(arg simple_collision_debug)">
       <xacro:rocker_stl_collision mesh_file="rocker_right_link.stl"/>
@@ -118,5 +116,5 @@
     <child link="rocker_right_link"/>
     <!-- Y: opprinnelig CAD/URDF (git). -->
-    <origin xyz="0.014227 -0.065999 0.021756" rpy="0 0 0"/>
+    <origin xyz="-0.014227 0.065999 0.021756" rpy="0 0 0"/>
     <axis xyz="0 1 0"/>
     <!-- Moderate URDF-demping + Gazebo-kontakt; unngaa for hoey friksjon som låser rocker-bogie. -->
@@ -146,5 +144,5 @@
       <parent link="base_link"/>
       <child link="feste_mellom_feste_og_stang_right_link"/>
-      <origin xyz="0.013913 -0.067245 0.076373" rpy="0 0 0"/>
+      <origin xyz="-0.013913 0.067245 0.076373" rpy="0 0 0"/>
       <axis xyz="1 0 0"/>
       <xacro:if value="$(arg enable_urdf_mimic)">
@@ -158,5 +156,5 @@
       <parent link="base_link"/>
       <child link="feste_mellom_feste_og_stang_right_link"/>
-      <origin xyz="0.013913 -0.067245 0.076373" rpy="0 0 0"/>
+      <origin xyz="-0.013913 0.067245 0.076373" rpy="0 0 0"/>
     </joint>
   </xacro:if>
@@ -182,5 +180,5 @@
       <parent link="feste_mellom_feste_og_stang_right_link"/>
       <child link="stang_right_link"/>
-      <origin xyz="-0.101730 -0.000140 0.000033" rpy="0 0 0"/>
+      <origin xyz="0.101730 0.000140 0.000033" rpy="0 0 0"/>
       <axis xyz="1 0 0"/>
       <xacro:if value="$(arg enable_urdf_mimic)">
@@ -194,5 +192,5 @@
       <parent link="feste_mellom_feste_og_stang_right_link"/>
       <child link="stang_right_link"/>
-      <origin xyz="-0.101730 -0.000140 0.000033" rpy="0 0 0"/>
+      <origin xyz="0.101730 0.000140 0.000033" rpy="0 0 0"/>
     </joint>
   </xacro:if>
@@ -218,5 +216,5 @@
       <parent link="base_link"/>
       <child link="feste_mellom_feste_og_stang_left_link"/>
-      <origin xyz="0.013977 0.064006 0.076371" rpy="0 0 0"/>
+      <origin xyz="-0.013977 -0.064006 0.076371" rpy="0 0 0"/>
       <xacro:if value="$(arg enable_urdf_mimic)">
         <mimic joint="rocker_bogie_diff_joint" multiplier="0.05" offset="0.0"/>
@@ -230,5 +228,5 @@
       <parent link="base_link"/>
       <child link="feste_mellom_feste_og_stang_left_link"/>
-      <origin xyz="0.013977 0.064006 0.076371" rpy="0 0 0"/>
+      <origin xyz="-0.013977 -0.064006 0.076371" rpy="0 0 0"/>
     </joint>
   </xacro:if>
@@ -253,5 +251,5 @@
       <parent link="feste_mellom_feste_og_stang_left_link"/>
       <child link="stang_left_link"/>
-      <origin xyz="-0.101903 0.001198 0.000110" rpy="0 0 0"/>
+      <origin xyz="0.101903 -0.001198 0.000110" rpy="0 0 0"/>
       <axis xyz="1 0 0"/>
       <xacro:if value="$(arg enable_urdf_mimic)">
@@ -265,5 +263,5 @@
       <parent link="feste_mellom_feste_og_stang_left_link"/>
       <child link="stang_left_link"/>
-      <origin xyz="-0.101903 0.001198 0.000110" rpy="0 0 0"/>
+      <origin xyz="0.101903 -0.001198 0.000110" rpy="0 0 0"/>
     </joint>
   </xacro:if>
@@ -279,7 +277,4 @@
       </material>
     </visual>
-    <xacro:if value="$(arg simple_collision_debug)">
-      <xacro:bogie_primitive_collision/>
-    </xacro:if>
     <xacro:unless value="$(arg simple_collision_debug)">
       <xacro:rocker_stl_collision mesh_file="bogie_right_link.stl"/>
@@ -296,5 +291,5 @@
     <child link="bogie_right_link"/>
     <!-- Origin = (gammel bogie-in-feste-frame) - (gammel rocker-in-feste-frame). -->
-    <origin xyz="0.087545 -0.025322 -0.050495" rpy="0 0 0"/>
+    <origin xyz="-0.087545 0.025322 -0.050495" rpy="0 0 0"/>
     <axis xyz="0 1 0"/>
     <dynamics damping="0.08" friction="0.015"/>
@@ -323,5 +318,5 @@
     <parent link="rocker_right_link"/>
     <child link="wheel_r1_link"/>
-    <origin xyz="-0.170916 -0.039688 -0.099612" rpy="0 0 0"/>
+    <origin xyz="0.170916 0.039688 -0.099612" rpy="0 0 0"/>
     <axis xyz="0 1 0"/>
     <dynamics damping="0.01" friction="0.0"/>
@@ -349,5 +344,5 @@
     <parent link="bogie_right_link"/>
     <child link="wheel_r2_link"/>
-    <origin xyz="-0.088585 -0.022644 -0.050672" rpy="0 0 0"/>
+    <origin xyz="0.088585 0.022644 -0.050672" rpy="0 0 0"/>
     <axis xyz="0 1 0"/>
     <dynamics damping="0.01" friction="0.0"/>
@@ -375,5 +370,5 @@
     <parent link="bogie_right_link"/>
     <child link="wheel_r3_link"/>
-    <origin xyz="0.081571 -0.016915 -0.048426" rpy="0 0 0"/>
+    <origin xyz="-0.081571 0.016915 -0.048426" rpy="0 0 0"/>
     <axis xyz="0 1 0"/>
     <dynamics damping="0.01" friction="0.0"/>
@@ -392,7 +387,4 @@
       </material>
     </visual>
-    <xacro:if value="$(arg simple_collision_debug)">
-      <xacro:rocker_primitive_collision/>
-    </xacro:if>
     <xacro:unless value="$(arg simple_collision_debug)">
       <xacro:rocker_stl_collision mesh_file="rocker_left_link.stl"/>
@@ -409,5 +401,5 @@
     <child link="rocker_left_link"/>
     <!-- Opprinnelig URDF (git). -->
-    <origin xyz="0.014252 0.064048 0.021830" rpy="0 0 0"/>
+    <origin xyz="-0.014252 -0.064048 0.021830" rpy="0 0 0"/>
     <axis xyz="0 1 0"/>
     <dynamics damping="0.10" friction="0.02"/>
@@ -428,7 +420,4 @@
       </material>
     </visual>
-    <xacro:if value="$(arg simple_collision_debug)">
-      <xacro:bogie_primitive_collision/>
-    </xacro:if>
     <xacro:unless value="$(arg simple_collision_debug)">
       <xacro:rocker_stl_collision mesh_file="bogie_left_link.stl"/>
@@ -444,5 +433,5 @@
     <parent link="rocker_left_link"/>
     <child link="bogie_left_link"/>
-    <origin xyz="0.087063 0.025935 -0.050644" rpy="0 0 0"/>
+    <origin xyz="-0.087063 -0.025935 -0.050645" rpy="0 0 0"/>
     <axis xyz="0 1 0"/>
     <dynamics damping="0.08" friction="0.015"/>
@@ -471,5 +460,5 @@
     <parent link="rocker_left_link"/>
     <child link="wheel_l1_link"/>
-    <origin xyz="-0.170218 0.040994 -0.100687" rpy="0 0 0"/>
+    <origin xyz="0.170218 -0.040994 -0.100687" rpy="0 0 0"/>
     <axis xyz="0 1 0"/>
     <dynamics damping="0.01" friction="0.0"/>
@@ -497,5 +486,5 @@
     <parent link="bogie_left_link"/>
     <child link="wheel_l2_link"/>
-    <origin xyz="-0.087657 0.020188 -0.050374" rpy="0 0 0"/>
+    <origin xyz="0.087657 -0.020188 -0.050374" rpy="0 0 0"/>
     <axis xyz="0 1 0"/>
     <dynamics damping="0.01" friction="0.0"/>
@@ -524,5 +513,5 @@
     <parent link="bogie_left_link"/>
     <child link="wheel_l3_link"/>
-    <origin xyz="0.082028 0.018253 -0.048351" rpy="0 0 0"/>
+    <origin xyz="-0.082028 -0.018253 -0.048350" rpy="0 0 0"/>
     <axis xyz="0 1 0"/>
     <dynamics damping="0.01" friction="0.0"/>
@@ -611,5 +600,5 @@
     <parent link="base_link"/>
     <child link="feste_rocker_karosseri_link"/>
-    <origin xyz="-0.091807 -0.001085 0.062183" rpy="0 0 0"/>
+    <origin xyz="0.091894 0.000000 0.061503" rpy="0 0 0"/>
   </joint>
   <link name="rocker_bogie_diff_link">
@@ -623,7 +612,4 @@
       </material>
     </visual>
-    <xacro:if value="$(arg simple_collision_debug)">
-      <xacro:diff_bar_primitive_collision/>
-    </xacro:if>
     <xacro:unless value="$(arg simple_collision_debug)">
       <xacro:rocker_stl_collision mesh_file="rocker_bogie_diff_link.stl"/>
@@ -684,5 +670,5 @@
     <parent link="feste_rocker_karosseri_link"/>
     <child link="rocker_bogie_diff_link"/>
-    <origin xyz="0.000012 0.000001 0.014" rpy="0 0 0"/>
+    <origin xyz="0.000109 0.001094 0.014506" rpy="0 0 0"/>
     <axis xyz="0 0 1"/>
     <!-- Diff-staven er lett; lav URDF-demping så plugin/terreng ikke konkurrerer. -->
@@ -714,5 +700,5 @@
     <parent link="base_link"/>
     <child link="tak_liten_link"/>
-    <origin xyz="0.100194 -0.000939 0.079219" rpy="0 0 0"/>
+    <origin xyz="-0.100194 0.000939 0.079219" rpy="0 0 0"/>
   </joint>
   <!-- =============================================================== -->
@@ -744,5 +730,5 @@
     <parent link="base_link"/>
     <child link="imu_link"/>
-    <origin xyz="0.001234 -0.000060 0.003194" rpy="0 0 0"/>
+    <origin xyz="-0.020281 0.000988 0.052512" rpy="0 0 0"/>
   </joint>
   <!-- === Stereokamera-hus (fronten av basen) === -->
@@ -776,5 +762,5 @@
     <child link="stereo_camera_link"/>
     <!-- CAD-opprinnelig posisjon fra Blender-prosjektet. Selve kamera-SENSOREN (Gazebo) festes direkte paa base_link med pose-offset i gz xacro-wrapperen, slik at hverken render- rekkefoelgen eller fixed-joint-lumping paavirker kamera- posen. Denne link-en er kun for visual mesh + TF. -->
-    <origin xyz="-0.166163 -0.008930 0.069183" rpy="0 0 0"/>
+    <origin xyz="0.165483 0.004944 0.068584" rpy="0 0 0"/>
   </joint>
   <!-- === Venstre kamera: fysisk frame + optisk frame === -->
@@ -790,5 +776,5 @@
     <parent link="stereo_camera_link"/>
     <child link="stereo_left_camera_link"/>
-    <origin xyz="-0.024178 0.024515 -0.006769" rpy="0 0 0"/>
+    <origin xyz="0.024178 -0.024515 -0.006769" rpy="0 0 0"/>
   </joint>
   <!-- Optisk frame: ROS-konvensjon (x=right, y=down, z=forward) rotert fra fysisk frame (x=forward, y=left, z=up) -->
@@ -811,5 +797,5 @@
     <parent link="stereo_camera_link"/>
     <child link="stereo_right_camera_link"/>
-    <origin xyz="-0.024077 -0.032034 -0.005843" rpy="0 0 0"/>
+    <origin xyz="0.024077 0.032034 -0.005843" rpy="0 0 0"/>
   </joint>
   <link name="stereo_right_optical_frame"/>
@@ -838,5 +824,5 @@
     <child link="depth_camera_optical_frame"/>
     <!-- ROS optical frame: x=right, y=down, z=forward -->
-    <origin xyz="-0.024258 -0.005494 -0.007196" rpy="-1.57079632679 0 -1.57079632679"/>
+    <origin xyz="0.024258 0.005494 -0.007196" rpy="-1.57079632679 0 -1.57079632679"/>
   </joint>
   <!-- =============================================================== -->
@@ -852,25 +838,4 @@
   <!-- Festet til rocker-linken slik at bracketen roterer med rockeren. -->
   <!-- === Hall-effekt-sensor (festet paa basen for rotasjonsmaaling) === -->
-  <link name="halleffekt_sensor_link">
-    <visual>
-      <origin xyz="0 0 0" rpy="0 0 0"/>
-      <geometry>
-        <mesh filename="package://moonmapper_description/meshes/visual/Hallefektsensor_link.stl" scale="1 1 1"/>
-      </geometry>
-      <material name="halleffekt_green">
-        <color rgba="0.1 0.6 0.2 1.0"/>
-      </material>
-    </visual>
-    <inertial>
-      <origin xyz="0 0 0" rpy="0 0 0"/>
-      <mass value="0.003"/>
-      <inertia ixx="1e-9" ixy="0" ixz="0" iyy="1e-9" iyz="0" izz="1e-9"/>
-    </inertial>
-  </link>
-  <joint name="halleffekt_sensor_joint" type="fixed">
-    <parent link="rocker_right_link"/>
-    <child link="halleffekt_sensor_link"/>
-    <origin xyz="-0.155776 -0.011745 -0.088736" rpy="0 0 0"/>
-  </joint>
   <!-- === Mikroskop (nede-pekende observasjonskamera) === -->
   <link name="mikroskop_link">
@@ -893,5 +858,5 @@
     <parent link="base_link"/>
     <child link="mikroskop_link"/>
-    <origin xyz="-0.091849 -0.001046 -0.006375" rpy="0 0 0"/>
+    <origin xyz="0.091849 0.001046 -0.006375" rpy="0 0 0"/>
   </joint>
   <!-- Optisk frame for mikroskop (ROS optical convention) -->
@@ -923,5 +888,5 @@
     <parent link="base_link"/>
     <child link="triad_sensor_1_link"/>
-    <origin xyz="-0.091911 0.046088 -0.043464" rpy="0 0 0"/>
+    <origin xyz="0.091911 -0.046088 -0.043464" rpy="0 0 0"/>
   </joint>
   <link name="triad_sensor_2_link">
@@ -944,5 +909,5 @@
     <parent link="base_link"/>
     <child link="triad_sensor_2_link"/>
-    <origin xyz="-0.091834 -0.048139 -0.043518" rpy="0 0 0"/>
+    <origin xyz="0.091833 0.048139 -0.043518" rpy="0 0 0"/>
   </joint>
 </robot>

File: src/moonmapper_description/urdf/moonmapper_rover_gazebo.urdf.xacro (robot description, xacro)
@@ -7,24 +7,47 @@
   <xacro:arg name="rocker_diff_debug" default="false"/>
   <xacro:arg name="rocker_diff_print_interval" default="0.5"/>
+  <!-- Friksjon/kontakt (overstyres av launch physics_profile). -->
+  <xacro:arg name="wheel_mu1" default="0.12"/>
+  <xacro:arg name="wheel_mu2" default="2.35"/>
+  <xacro:arg name="wheel_kp" default="9000.0"/>
+  <xacro:arg name="wheel_kd" default="55.0"/>
+  <xacro:arg name="wheel_use_fdir1" default="true"/>
   <!-- Grunnmodell: samme fil som RViz bruker (use_gazebo fra launch, typ. true) -->
   <xacro:include filename="$(find moonmapper_description)/urdf/moonmapper_rover.urdf.xacro"/>
-  <!-- Kontakt/friksjons-parametere for hjul. Hjul-link inkl. slatt motor-masse m~0,11 kg; base ~0,9 kg — moderate mu og avstemt kp/kd. -->
-  <xacro:property name="wheel_mu1" value="1.35"/>
-  <xacro:property name="wheel_mu2" value="1.15"/>
-  <!-- ODE bruker kp/kd for kontakt. Tyngre rover: litt lavere kp og avstemt kd gir stabil hjul-kontakt og rocker-bogie-artikulasjon. -->
-  <xacro:property name="wheel_kp" value="12000.0"/>
-  <xacro:property name="wheel_kd" value="40.0"/>
-  <!-- Macro: kontakt-/friksjons-parametere for hjul-link -->
+  <!-- Macro: kontakt-/friksjons-parametere for hjul-link (akse Y = rulling, mu2 = tverrgrep). -->
   <xacro:macro name="wheel_gazebo" params="link">
     <gazebo reference="${link}">
-      <mu1>${wheel_mu1}</mu1>
-      <mu2>${wheel_mu2}</mu2>
-      <kp>${wheel_kp}</kp>
-      <kd>${wheel_kd}</kd>
+      <mu1>$(arg wheel_mu1)</mu1>
+      <mu2>$(arg wheel_mu2)</mu2>
+      <kp>$(arg wheel_kp)</kp>
+      <kd>$(arg wheel_kd)</kd>
       <minDepth>0.0005</minDepth>
-      <!-- Ikke klipp kontakt-korrigering for lavt; 0.5 m/s ga ofte «fast» hjul med bullet. -->
       <maxVel>25.0</maxVel>
-      <!-- Ingen fdir1: anisotrop friksjon kan motvirke ren rulling rundt Y-akse. -->
+      <xacro:if value="$(arg wheel_use_fdir1)">
+        <fdir1>0 1 0</fdir1>
+      </xacro:if>
       <selfCollide>false</selfCollide>
+      <!-- Gazebo Sim/DART: eksplisitt surface/ode i tillegg til legacy mu1/mu2. -->
+      <surface>
+        <friction>
+          <ode>
+            <mu>$(arg wheel_mu2)</mu>
+            <mu2>$(arg wheel_mu2)</mu2>
+            <slip1>0.0</slip1>
+            <slip2>0.0</slip2>
+            <xacro:if value="$(arg wheel_use_fdir1)">
+              <fdir1>0 1 0</fdir1>
+            </xacro:if>
+          </ode>
+        </friction>
+        <contact>
+          <ode>
+            <kp>$(arg wheel_kp)</kp>
+            <kd>$(arg wheel_kd)</kd>
+            <min_depth>0.0005</min_depth>
+            <max_vel>25.0</max_vel>
+          </ode>
+        </contact>
+      </surface>
     </gazebo>
   </xacro:macro>
