Commit message: chore: remove UWB/Nav2 experiment; sim_rover_clean; ekf_wheel in description
Co-authored-by: Cursor <cursoragent@cursor.com>

File: src/moonmapper_description/urdf/moonmapper_rover.urdf.xacro (robot description, xacro)
@@ -782,17 +782,4 @@
     <origin xyz="0.001234 -0.000060 0.003194" rpy="0 0 0"/>
   </joint>
-  <!-- === UWB/BU04-tag (statisk frame for digital tvilling / trilateration) === -->
-  <link name="uwb_tag_link">
-    <inertial>
-      <origin xyz="0 0 0" rpy="0 0 0"/>
-      <mass value="0.001"/>
-      <inertia ixx="1e-9" ixy="0" ixz="0" iyy="1e-9" iyz="0" izz="1e-9"/>
-    </inertial>
-  </link>
-  <joint name="uwb_tag_joint" type="fixed">
-    <parent link="base_link"/>
-    <child link="uwb_tag_link"/>
-    <origin xyz="0 0 0.10" rpy="0 0 0"/>
-  </joint>
   <!-- === Stereokamera-hus (fronten av basen) === -->
   <!-- Mesh er ~4x13x4 mm, oppgitt i meter. Plasseres paa fronten av basen, litt over toppen. -->

Commit message: fix(physics): skid-steer baseline — én cmd_vel-vei, +1 sign, hjul-sylinder
- Fjernet ROS_TO_GZ /cmd_vel-bro (ros_gz_bridge.yaml); unngår parallell styring mot gz_ros2_control.
- cmd_vel_odom_relay: standard cmd_linear_x_sign=+1, frame_id=base_footprint, oppdatert docstring.
- gazebo_rover: launch-arg cmd_vel_relay_frame_id, cmd_linear_x_sign default 1.0, motorvei dokumentert i toppkommentar.
- URDF: base_footprint uten inertial; alle seks hjul bruker sylinder-kollisjon langs felles akse (Y).
- Gazebo xacro: litt høyere hjul-friksjon (mu1/mu2) for yaw-moment ved skid-steer.
- tools/test_drive_sanity.sh: A/B/C cmd_vel-sekvens for manuell verifikasjon i Gazebo.

Co-authored-by: Cursor <cursoragent@cursor.com>

File: src/moonmapper_description/urdf/moonmapper_rover.urdf.xacro (robot description, xacro)
@@ -9,5 +9,5 @@
   <xacro:arg name="enable_urdf_mimic" default="true"/>
   <xacro:arg name="use_gazebo" default="false"/>
-  <!-- Enkle primitiver for rocker/bogie/hjul i stedet for STL (mindre «krok» mot bakken). -->
+  <!-- Enkle primitiver for rocker/bogie i stedet for STL (mindre «krok» mot bakken). Hjul bruker alltid sylinder-kollisjon. -->
   <xacro:arg name="simple_collision_debug" default="false"/>
   <xacro:macro name="rocker_stl_collision" params="mesh_file">
@@ -52,12 +52,6 @@
     </collision>
   </xacro:macro>
-  <!-- Base footprint: bakkeplan under rover (Nav2/MPPI). Lett rot-node; unngaa null-inertia i Gazebo. -->
-  <link name="base_footprint">
-    <inertial>
-      <origin xyz="0 0 0" rpy="0 0 0"/>
-      <mass value="0.0001"/>
-      <inertia ixx="1e-12" ixy="0" ixz="0" iyy="1e-12" iyz="0" izz="1e-12"/>
-    </inertial>
-  </link>
+  <!-- base_footprint: masseløst root-frame (REP-105). Masse, treghet og chassis-kollisjon ligger på base_link. -->
+  <link name="base_footprint"/>
   <joint name="base_footprint_to_base_link" type="fixed">
     <parent link="base_footprint"/>
@@ -318,10 +312,5 @@
       </material>
     </visual>
-    <xacro:if value="$(arg simple_collision_debug)">
-      <xacro:wheel_primitive_collision/>
-    </xacro:if>
-    <xacro:unless value="$(arg simple_collision_debug)">
-      <xacro:rocker_stl_collision mesh_file="wheel_r1_link.stl"/>
-    </xacro:unless>
+    <xacro:wheel_primitive_collision/>
     <inertial>
       <!-- Hjul 0,048 kg + tidl. motor 0,062 kg slatt inn i hjullink (ingen motor_*); sylinder om Y, r=0,045, w=0,039, m=0,11. -->
@@ -349,10 +338,5 @@
       </material>
     </visual>
-    <xacro:if value="$(arg simple_collision_debug)">
-      <xacro:wheel_primitive_collision/>
-    </xacro:if>
-    <xacro:unless value="$(arg simple_collision_debug)">
-      <xacro:rocker_stl_collision mesh_file="wheel_r2_link.stl"/>
-    </xacro:unless>
+    <xacro:wheel_primitive_collision/>
     <inertial>
       <!-- Hjul 0,048 kg + tidl. motor 0,062 kg slatt inn i hjullink (ingen motor_*); sylinder om Y, r=0,045, w=0,039, m=0,11. -->
@@ -380,10 +364,5 @@
       </material>
     </visual>
-    <xacro:if value="$(arg simple_collision_debug)">
-      <xacro:wheel_primitive_collision/>
-    </xacro:if>
-    <xacro:unless value="$(arg simple_collision_debug)">
-      <xacro:rocker_stl_collision mesh_file="wheel_r3_link.stl"/>
-    </xacro:unless>
+    <xacro:wheel_primitive_collision/>
     <inertial>
       <!-- Hjul 0,048 kg + tidl. motor 0,062 kg slatt inn i hjullink (ingen motor_*); sylinder om Y, r=0,045, w=0,039, m=0,11. -->
@@ -481,10 +460,5 @@
       </material>
     </visual>
-    <xacro:if value="$(arg simple_collision_debug)">
-      <xacro:wheel_primitive_collision/>
-    </xacro:if>
-    <xacro:unless value="$(arg simple_collision_debug)">
-      <xacro:rocker_stl_collision mesh_file="wheel_l1_link.stl"/>
-    </xacro:unless>
+    <xacro:wheel_primitive_collision/>
     <inertial>
       <!-- Hjul 0,048 kg + tidl. motor 0,062 kg slatt inn i hjullink (ingen motor_*); sylinder om Y, r=0,045, w=0,039, m=0,11. -->
@@ -512,10 +486,5 @@
       </material>
     </visual>
-    <xacro:if value="$(arg simple_collision_debug)">
-      <xacro:wheel_primitive_collision/>
-    </xacro:if>
-    <xacro:unless value="$(arg simple_collision_debug)">
-      <xacro:rocker_stl_collision mesh_file="wheel_l2_link.stl"/>
-    </xacro:unless>
+    <xacro:wheel_primitive_collision/>
     <inertial>
       <!-- Hjul 0,048 kg + tidl. motor 0,062 kg slatt inn i hjullink (ingen motor_*); sylinder om Y, r=0,045, w=0,039, m=0,11. -->
@@ -543,10 +512,5 @@
       </material>
     </visual>
-    <xacro:if value="$(arg simple_collision_debug)">
-      <xacro:wheel_primitive_collision/>
-    </xacro:if>
-    <xacro:unless value="$(arg simple_collision_debug)">
-      <xacro:rocker_stl_collision mesh_file="wheel_l3_link.stl"/>
-    </xacro:unless>
+    <xacro:wheel_primitive_collision/>
     <inertial>
       <!-- Hjul 0,048 kg + tidl. motor 0,062 kg slatt inn i hjullink (ingen motor_*); sylinder om Y, r=0,045, w=0,039, m=0,11. -->

File: src/moonmapper_description/urdf/moonmapper_rover_gazebo.urdf.xacro (robot description, xacro)
@@ -10,6 +10,6 @@
   <xacro:include filename="$(find moonmapper_description)/urdf/moonmapper_rover.urdf.xacro"/>
   <!-- Kontakt/friksjons-parametere for hjul. Hjul-link inkl. slatt motor-masse m~0,11 kg; base ~0,9 kg — moderate mu og avstemt kp/kd. -->
-  <xacro:property name="wheel_mu1" value="1.15"/>
-  <xacro:property name="wheel_mu2" value="1.0"/>
+  <xacro:property name="wheel_mu1" value="1.35"/>
+  <xacro:property name="wheel_mu2" value="1.15"/>
   <!-- ODE bruker kp/kd for kontakt. Tyngre rover: litt lavere kp og avstemt kd gir stabil hjul-kontakt og rocker-bogie-artikulasjon. -->
   <xacro:property name="wheel_kp" value="12000.0"/>

Commit message: Fix sim physics regression and align camera frames with autonomy.
Restore wheel collision cylinder orientation, match stereo/depth URDF to
Gazebo sensor poses, publish /scan in depth_camera_optical_frame, and add
frontier goal commitment plus explored-area memory for stable V1 exploration.

Co-authored-by: Cursor <cursoragent@cursor.com>

File: src/moonmapper_description/urdf/moonmapper_rover.urdf.xacro (robot description, xacro)
@@ -11,4 +11,12 @@
   <!-- simple_collision_debug: kun hjul har kollisjon (ingen rocker/bogie/diff-bar) — anbefalt for Gazebo 6WD-traksjon. -->
   <xacro:arg name="simple_collision_debug" default="false"/>
+  <!-- Gazebo urdf2sdf krever inertial på alle links; bruk på TF-only kamera-frames. -->
+  <xacro:macro name="negligible_inertial">
+    <inertial>
+      <origin xyz="0 0 0" rpy="0 0 0"/>
+      <mass value="1e-6"/>
+      <inertia ixx="1e-12" ixy="0" ixz="0" iyy="1e-12" iyz="0" izz="1e-12"/>
+    </inertial>
+  </xacro:macro>
   <xacro:macro name="rocker_stl_collision" params="mesh_file">
     <collision>
@@ -73,6 +81,6 @@
     <xacro:unless value="$(arg simple_collision_debug)">
     <collision>
-      <!-- Primitiv boks, forskjøvet +X/+Z: front (kamera) er ca. -X; boks bakover/opp unngar at underkant tar bakken før hjulene finner likevekt. -->
-      <origin xyz="0.020 0 0.011" rpy="0 0 0"/>
+      <!-- Primitiv boks, forskjøvet −X/+Z: front (stereo) er ca. +X; boks bakover/opp unngår at underkant tar bakken før hjulene finner likevekt. -->
+      <origin xyz="-0.020 0 0.011" rpy="0 0 0"/>
       <geometry>
         <box size="0.048 0.025 0.018"/>
@@ -81,5 +89,5 @@
     </xacro:unless>
     <!-- Gazebo krever inertial paa enhver dynamisk link. Målt masse 0,907 kg; treghet homogen boks 0,305×0,105×0,110 m (ixx=(1/12)m(y²+z²) osv.). -->
-    <!-- ADVARSEL: -X er mot FRONT (stereo ~ -0.166 m). Aldri sett base_link inertial x negativ for aa «løfte nesa» — det flytter masse FOROVER. -->
+    <!-- ADVARSEL: +X er mot FRONT (stereo ~ +0.166 m). Aldri sett base_link inertial x negativ for å «løfte nesa» — det flytter masse BAKOVER. -->
     <inertial>
       <origin xyz="0.038 0 0.010" rpy="0 0 0"/>
@@ -106,5 +114,5 @@
     <inertial>
       <!-- Målt 0,166 kg/stk; treghet estimert som homogen boks = rocker_primitive_collision (0,16×0,042×0,042 m). -->
-      <!-- Hjul l1 ligger ca. -0.16 m i X fra pivot; uten offset blir rocker for «tung» foran. Liten +X flytter rapportert CoM mot bogie (+X = bak langs armen). -->
+      <!-- Hjul l1 ligger ca. -0.16 m i X fra pivot; uten offset blir rocker for «tung» foran. Liten +X flytter rapportert CoM mot bogie (−X = bak langs armen). -->
       <origin xyz="0.030 0 -0.028" rpy="0 0 0"/>
       <mass value="0.166"/>
@@ -744,17 +752,25 @@
       </material>
     </visual>
-    <xacro:unless value="$(arg simple_collision_debug)">
-    <collision>
-      <origin xyz="0 0 0" rpy="0 0 0"/>
-      <geometry>
-        <mesh filename="package://moonmapper_description/meshes/visual/steriokamera_link.stl" scale="1 1 1"/>
-      </geometry>
-    </collision>
+    <!-- Ingen kollisjon i Gazebo; sensorer festes på base_link (gz-xacro). -->
+    <xacro:unless value="$(arg use_gazebo)">
+      <xacro:unless value="$(arg simple_collision_debug)">
+        <collision>
+          <origin xyz="0 0 0" rpy="0 0 0"/>
+          <geometry>
+            <mesh filename="package://moonmapper_description/meshes/visual/steriokamera_link.stl" scale="1 1 1"/>
+          </geometry>
+        </collision>
+      </xacro:unless>
     </xacro:unless>
-    <inertial>
-      <origin xyz="0 0 0" rpy="0 0 0"/>
-      <mass value="0.002"/>
-      <inertia ixx="2e-7" ixy="0" ixz="0" iyy="2e-7" iyz="0" izz="2e-7"/>
-    </inertial>
+    <xacro:if value="$(arg use_gazebo)">
+      <xacro:negligible_inertial/>
+    </xacro:if>
+    <xacro:unless value="$(arg use_gazebo)">
+      <inertial>
+        <origin xyz="0 0 0" rpy="0 0 0"/>
+        <mass value="0.002"/>
+        <inertia ixx="2e-7" ixy="0" ixz="0" iyy="2e-7" iyz="0" izz="2e-7"/>
+      </inertial>
+    </xacro:unless>
   </link>
   <joint name="stereo_camera_joint" type="fixed">
@@ -762,40 +778,32 @@
     <child link="stereo_camera_link"/>
     <!-- CAD-opprinnelig posisjon fra Blender-prosjektet. Selve kamera-SENSOREN (Gazebo) festes direkte paa base_link med pose-offset i gz xacro-wrapperen, slik at hverken render- rekkefoelgen eller fixed-joint-lumping paavirker kamera- posen. Denne link-en er kun for visual mesh + TF. -->
+    <!-- Front = +X i base_link (REP-103). π rundt Z speiler CAD-mesh slik at huset sitter på nesa. -->
     <origin xyz="0.165483 0.004944 0.068584" rpy="0 0 0"/>
   </joint>
   <!-- === Venstre kamera: fysisk frame + optisk frame === -->
   <!-- Venstre = +y (ROS: +y peker til venstre) -->
+  <!-- === Venstre kamera === -->
   <link name="stereo_left_camera_link">
-    <inertial>
-      <origin xyz="0 0 0" rpy="0 0 0"/>
-      <mass value="0.001"/>
-      <inertia ixx="1e-9" ixy="0" ixz="0" iyy="1e-9" iyz="0" izz="1e-9"/>
-    </inertial>
+    <xacro:negligible_inertial/>
   </link>
   <joint name="stereo_left_camera_joint" type="fixed">
     <parent link="stereo_camera_link"/>
     <child link="stereo_left_camera_link"/>
-    <origin xyz="0.024178 -0.024515 -0.006769" rpy="0 0 0"/>
-  </joint>
-  <!-- Optisk frame: ROS-konvensjon (x=right, y=down, z=forward) rotert fra fysisk frame (x=forward, y=left, z=up) -->
+    <origin xyz="0.032910 0.034100 0.002791" rpy="0 0 0"/>
+  </joint>
   <link name="stereo_left_optical_frame"/>
   <joint name="stereo_left_optical_joint" type="fixed">
     <parent link="stereo_left_camera_link"/>
     <child link="stereo_left_optical_frame"/>
-    <!-- ROS optical frame: x=right, y=down, z=forward -->
-    <origin xyz="-0.024178 0.024515 -0.006769" rpy="-1.57079632679 0 -1.57079632679"/>
-  </joint>
-  <!-- === Hoeyre kamera === -->
+    <origin xyz="0 0 0" rpy="-1.57079632679 0 -1.57079632679"/>
+  </joint>
+  <!-- === Høyre kamera === -->
   <link name="stereo_right_camera_link">
-    <inertial>
-      <origin xyz="0 0 0" rpy="0 0 0"/>
-      <mass value="0.001"/>
-      <inertia ixx="1e-9" ixy="0" ixz="0" iyy="1e-9" iyz="0" izz="1e-9"/>
-    </inertial>
+    <xacro:negligible_inertial/>
   </link>
   <joint name="stereo_right_camera_joint" type="fixed">
     <parent link="stereo_camera_link"/>
     <child link="stereo_right_camera_link"/>
-    <origin xyz="0.024077 0.032034 -0.005843" rpy="0 0 0"/>
+    <origin xyz="0.032910 -0.032034 0.002791" rpy="0 0 0"/>
   </joint>
   <link name="stereo_right_optical_frame"/>
@@ -803,19 +811,14 @@
     <parent link="stereo_right_camera_link"/>
     <child link="stereo_right_optical_frame"/>
-    <!-- ROS optical frame: x=right, y=down, z=forward -->
-    <origin xyz="-0.024077 -0.032034 -0.005843" rpy="-1.57079632679 0 -1.57079632679"/>
+    <origin xyz="0 0 0" rpy="-1.57079632679 0 -1.57079632679"/>
   </joint>
   <!-- ====== Depth / RGB-D-kamera ====== Samme fysisk hus som stereokameraet, sentrert midt mellom venstre og hoeyre RGB-sensor. Ren TF-link; Gazebo-sensoren festes direkte paa base_link med <pose> (se gz-xacro). -->
   <link name="depth_camera_link">
-    <inertial>
-      <origin xyz="0 0 0" rpy="0 0 0"/>
-      <mass value="0.001"/>
-      <inertia ixx="1e-9" ixy="0" ixz="0" iyy="1e-9" iyz="0" izz="1e-9"/>
-    </inertial>
+    <xacro:negligible_inertial/>
   </link>
   <joint name="depth_camera_joint" type="fixed">
     <parent link="stereo_camera_link"/>
     <child link="depth_camera_link"/>
-    <origin xyz="-0.024258 -0.005494 -0.007196" rpy="0 0 0"/>
+    <origin xyz="0.039709 0.002014 0.002791" rpy="0 0 0"/>
   </joint>
   <link name="depth_camera_optical_frame"/>
@@ -824,5 +827,5 @@
     <child link="depth_camera_optical_frame"/>
     <!-- ROS optical frame: x=right, y=down, z=forward -->
-    <origin xyz="0.024258 0.005494 -0.007196" rpy="-1.57079632679 0 -1.57079632679"/>
+    <origin xyz="0 0 0" rpy="-1.57079632679 0 -1.57079632679"/>
   </joint>
   <!-- =============================================================== -->
@@ -866,5 +869,5 @@
     <child link="mikroskop_optical_frame"/>
     <!-- ROS optical frame: x=right, y=down, z=forward -->
-    <origin xyz="0 0 0" rpy="-1.57079632679 0 -1.57079632679"/>
+    <origin xyz="0 0 0" rpy="-0 0 -0"/>
   </joint>
   <!-- === Triad-sensorer (magnetometer/solvektor) === -->

File: src/moonmapper_description/urdf/moonmapper_rover_gazebo.urdf.xacro (robot description, xacro)
@@ -251,11 +251,11 @@
   <!-- URDF positions (base_link frame): -->
   <!-- imu_link: ( 0.001234, -0.000060, 0.003194) -->
-  <!-- stereo_camera_link: (-0.166163, -0.008930, 0.069183) -->
-  <!-- stereo_left_camera_link: (-0.190341, 0.015585, 0.062414) -->
-  <!-- stereo_right_camera_link:(-0.190240, -0.040964, 0.063340) -->
-  <!-- depth_camera_link: (-0.190421, -0.014424, 0.061987) -->
-  <!-- mikroskop_link: (-0.091849,-0.001046,-0.006375) -->
-  <!-- triad_sensor_1_link: (-0.091911, 0.046088,-0.043464) -->
-  <!-- triad_sensor_2_link: (-0.091834,-0.048139,-0.043518) -->
+  <!-- Gazebo Sim renderer langs sensor +X (ikke ROS optical +Z). Posisjon = URDF optical origin; rpy 0 0 0 => +X base = rett frem. -->
+  <!-- stereo_left_optical_frame:  ( 0.198393,  0.039044, 0.071375) -->
+  <!-- stereo_right_optical_frame: ( 0.198393, -0.027090, 0.071375) -->
+  <!-- depth_camera_optical_frame: ( 0.205192,  0.006958, 0.071375) -->
+  <!-- mikroskop_link: ( 0.091849, 0.001046,-0.006375) -->
+  <!-- triad_sensor_1_link: ( 0.091911,-0.046088,-0.043464) -->
+  <!-- triad_sensor_2_link: ( 0.091833, 0.048139,-0.043518) -->
   <!-- halleffekt_sensor_link: festet på rocker_right_link (URDF) -->
   <!-- =============================================================== -->
@@ -311,8 +311,7 @@
       </imu>
     </sensor>
-    <!-- === Venstre kamera (peker +X i base-frame) === Oppløsning 320x240 for aa la GPU-en klare begge kameraer; oek til 640x480 naar GPU er ledig. -->
+    <!-- === Venstre kamera (pos = URDF optical; gz +X = fremover i base_link) === -->
     <sensor name="stereo_left_camera" type="camera">
-      <!-- Rotate 180deg yaw so camera faces +X in base_link -->
-      <pose>-0.190341 0.015585 0.062414 0 0 3.14159</pose>
+      <pose>0.198393 0.039044 0.071375 0 0 0</pose>
       <always_on>true</always_on>
       <update_rate>15</update_rate>
@@ -341,6 +340,5 @@
     <!-- === Hoeyre kamera === -->
     <sensor name="stereo_right_camera" type="camera">
-      <!-- Rotate 180deg yaw so camera faces +X in base_link -->
-      <pose>-0.190240 -0.040964 0.063340 0 0 3.14159</pose>
+      <pose>0.198393 -0.027090 0.071375 0 0 0</pose>
       <always_on>true</always_on>
       <update_rate>15</update_rate>
@@ -368,6 +366,5 @@
     <!-- === RGB-D / Depth-kamera === type="rgbd_camera" publiserer RGB-bilde, depth-bilde OG point cloud samtidig. Plassert midt mellom de to stereo- sensorene (y=0) paa samme hoeyde. Topics fra gz-sim (med <topic>depth_camera</topic>): /depth_camera/image (gz.msgs.Image) /depth_camera/depth_image (gz.msgs.Image, 32FC1) /depth_camera/points (gz.msgs.PointCloudPacked) /depth_camera/camera_info (gz.msgs.CameraInfo) Near-planet er hardt begrenset til 0.1 m paa moderne GPU- rendere (ogre2), sa vi setter 0.05 -> clampes til 0.1. Den er lav nok for roveren vaar. -->
     <sensor name="depth_camera" type="rgbd_camera">
-      <!-- Rotate 180deg yaw so camera faces +X in base_link -->
-      <pose>-0.190421 -0.014424 0.061987 0 0 3.14159</pose>
+      <pose>0.205192 0.006958 0.071375 0 0 0</pose>
       <always_on>true</always_on>
       <update_rate>15</update_rate>
@@ -398,5 +395,5 @@
     <sensor name="microscope_camera" type="camera">
       <!-- base_link -> mikroskop_link (samme xyz som URDF mikroskop_joint). -->
-      <pose>-0.091849 -0.001046 -0.006375 0 1.57079632679 0</pose>
+      <pose>0.091849 0.001046 -0.006375 0 0 0</pose>
       <always_on>true</always_on>
       <update_rate>10</update_rate>
@@ -424,5 +421,5 @@
     </sensor>
   </gazebo>
-  <!-- Kamerahuset er ren visual; la den lumpes som vanlig med base_link -->
+  <!-- Kameratre: negligible inertial + lumping inn i base_link (urdf2sdf-krav). Ingen kollisjon. -->
   <gazebo reference="stereo_camera_link">
     <selfCollide>false</selfCollide>
